Commit message: pushing new stuff

File: src/mybot_description/urdf/mybot.xacro (robot description, xacro)
@@ -137,5 +137,5 @@
     <joint_properties damping="1.0" friction="1.0"/>
   </joint>
-  <link name="camera">
+  <!--link name="camera">
     <collision>
       <origin xyz="0 0 0" rpy="0 0 0"/>
@@ -163,13 +163,13 @@
     <parent link="chassis"/>
     <child link="camera"/>
-  </joint>
-  <joint name="hokuyo_joint" type="fixed">
+  </joint-->
+  <joint name="rplidar_joint" type="fixed">
     <axis xyz="0 1 0" />
     <origin xyz=".15 0 .1" rpy="0 0 0"/>
     <parent link="chassis"/>
-    <child link="hokuyo"/>
+    <child link="rplidar"/>
   </joint>
   <!-- Hokuyo Laser -->
-  <link name="hokuyo">
+  <link name="rplidar">
     <collision>
       <origin xyz="0 0 0" rpy="0 0 0"/>

Commit message: update

File: src/mybot_description/urdf/mybot.xacro (robot description, xacro)
@@ -137,5 +137,5 @@
     <joint_properties damping="1.0" friction="1.0"/>
   </joint>
-  <!--link name="camera">
+  <link name="camera">
     <collision>
       <origin xyz="0 0 0" rpy="0 0 0"/>
@@ -163,13 +163,13 @@
     <parent link="chassis"/>
     <child link="camera"/>
-  </joint-->
-  <joint name="rplidar_joint" type="fixed">
+  </joint>
+  <joint name="hokuyo_joint" type="fixed">
     <axis xyz="0 1 0" />
     <origin xyz=".15 0 .1" rpy="0 0 0"/>
     <parent link="chassis"/>
-    <child link="rplidar"/>
+    <child link="hokuyo"/>
   </joint>
   <!-- Hokuyo Laser -->
-  <link name="rplidar">
+  <link name="hokuyo">
     <collision>
       <origin xyz="0 0 0" rpy="0 0 0"/>
